File: Hardware/Gateway/Gateway.kicad_sch (KiCad schematic)
At the start: 10 parts, among them Q1 AO3401A, SW1 SW_Push, SW2 SW_Push, U1 ESP32-C3, U2 Mini560

Commit message: docs(wiring diagram): Doorlock and Gateway Ver. 1
Parts:
- added C5, C6: 100nF, symbol Device:C
- SW1: value SW_Push -> WiFi Config
- SW2: value SW_Push -> ESPNOW Config
Connections:
- net GND: now also C5.2, C6.2
- net at SW1.2, U1.7 (GPIO20): now also C5.1
- net at SW2.2, U1.8 (GPIO21): now also C6.1
Other:
- moved on the sheet: SW1, SW2
