File: Hardware/Doorlock/Doorlock.kicad_sch (KiCad schematic)
At the start: 22 parts, among them J1 Doorlock Module, J2 Motor Servo, Q1 AO3401A, Q2 AO3401A, SW1 Reset Button, U1 Mini560, U2 ESP32-C3, U3 DRV8833

Commit message: feat(hardware): Revisi rangkaian indikator baterai.
Co-Authored-By: Claude Opus 5.5 <noreply@anthropic.com>
Parts:
- removed C6: 100nF, symbol Device:C
- removed J2: Motor Servo, symbol Connector:Conn_01x02_Pin
- added J2: Mortise, symbol Connector:Conn_01x08_Pin
- added Q3: NPN, symbol Simulation_SPICE:NPN
- added R8: 100kΩ, symbol Device:R
Connections:
- net BAT_EN: now also U2.8 (GPIO21), R8.1; no longer Q2.1 (G), R5.2, U2.7 (GPIO20)
- net BAT_IND: now also U2.13 (GPIO4/ADC1/SDA); no longer U2.12 (GPIO3)
- net GND: now also J1.3 (Pin_3), J1.7 (Pin_7), J2.2 (Pin_2), J2.6 (Pin_6), Q3.3 (E); no longer J1.2 (Pin_2), J1.6 (Pin_6)
- net K: now also J2.3 (Pin_3); no longer J1.3 (Pin_3)
- net L: now also J2.5 (Pin_5); no longer J1.5 (Pin_5)
- net M+: now also J1.2 (Pin_2); no longer J1.7 (Pin_7)
- net M-: now also J1.1 (Pin_1); no longer J1.8 (Pin_8)
- net O: now also J2.4 (Pin_4); no longer J1.4 (Pin_4)
- net VCC: now also J1.8 (Pin_8); no longer J1.1 (Pin_1)
- net M_OUT1: now reaches C7.2, U3.11 (OUT1)
- net M_OUT1: now also J2.7 (Pin_7)
- net M_OUT2: now reaches C7.1, U3.10 (OUT2)
- net M_OUT2: now also J2.8 (Pin_8)
- net at SW1.2: now also U2.7 (GPIO20); no longer U2.8 (GPIO21)
- new net: Q3.2 (B), R8.2
- new net: Q2.1 (G), Q3.1 (C), R5.2
- new net 7,5V: J2.1 (Pin_1)
- no-connect marks 0 -> 3

Commit message: feat(hardware): Revisi divider M+/M- dan indikator baterai.
Divider M+/M- jadi 200k/100k (rasio 3), R6 indikator baterai jadi 200k, dan label M+/M- di konektor Doorlock Module ditukar sesuai wiring.

Co-Authored-By: Claude Opus 5.5 <noreply@anthropic.com>
Parts:
- R1, R3: value 100kΩ -> 200kΩ
- R2, R4: value 180kΩ -> 100kΩ
- R6: value 180kΩ -> 200kΩ
Connections:
- net M+: now also J1.1 (Pin_1); no longer J1.2 (Pin_2)
- net M-: now also J1.2 (Pin_2); no longer J1.1 (Pin_1)
Changed lines of the file:
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@@
 		)
 	)
-	(label "M+"
+	(label "M-"
 		(at 52.07 77.47 0)
 		(effects
@@
 		)
 	)
-	(label "M-"
+	(label "M+"
 		(at 52.07 74.93 0)
 		(effects
@@
 			)
 		)
-		(property "Value" "180kΩ"
+		(property "Value" "200kΩ"
 			(at 60.96 173.9899 0)
 			(show_name no)
@@
 			)
 		)
-		(property "Value" "180kΩ"
+		(property "Value" "100kΩ"
 			(at 200.66 97.7899 0)
 			(show_name no)
@@
 			)
 		)
-		(property "Value" "100kΩ"
+		(property "Value" "200kΩ"
 			(at 204.47 105.41 90)
 			(show_name no)
@@
 			)
 		)
-		(property "Value" "180kΩ"
+		(property "Value" "100kΩ"
 			(at 217.17 101.5999 0)
 			(show_name no)
@@
 			)
 		)
-		(property "Value" "100kΩ"
+		(property "Value" "200kΩ"
 			(at 220.98 110.49 90)
 			(show_name no)
